File: Aux Power Supply V5.kicad_sch (KiCad schematic)
At the start: 208 parts, among them IC1 ACS780LLRTR-050U-T, IC2 ACS780LLRTR-050U-T, J1 Screw_Terminal_01x01, J10 Screw_Terminal_01x01, J11 Screw_Terminal_01x01, J12 I_Sense_R, J2 Screw_Terminal_01x01, J3 I_Sense_R, J4 Conn_01x05, J5 5499923-4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

Commit message: changed bypass cap values to correct vals
Parts:
- C36: value 4.7uf -> 10uF
Changed lines of the file:
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@@
       (effects (font (size 1.27 1.27)) (justify left))
     )
-    (property "Value" "4.7uf" (at 214.63 119.38 0)
+    (property "Value" "10uF" (at 214.63 119.38 0)
       (effects (font (size 1.27 1.27)) (justify left))
     )

Commit message: updated documentation
Parts:
- removed C51, C53, C54, C57: 0.1uf, Capacitor_SMD:C_1206_3216Metric_Pad1.33x1.80mm_HandSolder, symbol Device:C_Small
- added C51, C53, C54, C55: 10uF, Capacitor_SMD:C_0805_2012Metric_Pad1.18x1.45mm_HandSolder, symbol SBS-ChargerV5-rescue:C_Small-Device-2-channel-half-bridge-rescue-SBS-charger-re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
- C22, C23, C24, C25, C34, C35, C37: value 4.7uf -> 10uF
Connections:
- net +18V_BOT_T1: now also C53.2
- net +18V_BOT_T2: now also C34.1, C55.2; no longer C37.1
- net +18V_TOP_T1: now also C37.1, C51.2; no longer C34.1
- net +18V_TOP_T2: now also C54.2
- net KELV_BOT_T1: now also C53.1
- net KELV_BOT_T2: now also C34.2, C55.1; no longer C37.2
- net KELV_TOP_T1: now also C37.2, C51.1; no longer C34.2
- net KELV_TOP_T2: now also C54.1
