File: Aux Power Supply V5.kicad_pcb (KiCad board)
At the start: 4 copper layers, 253 x 160 mm, 208 parts, among them IC1 ACS780LLRTR-050U-T, IC2 ACS780LLRTR-050U-T, J1 Screw_Terminal_01x01, J10 Screw_Terminal_01x01, J11 Screw_Terminal_01x01, J12 I_Sense_R, J2 Screw_Terminal_01x01, J3 I_Sense_R, J4 Conn_01x05, J5 5499923-4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

Commit message: locked PCB editor
Other:
- board text added: "locked"
- board text removed: "+5V"
- board text removed: "."
- board text removed: "AUX POWER SUPPLY V5"
- board text removed: "DC_IN"
- board text removed: "DC_OUT"
- board text removed: "GATE"
- board text removed: "GND"
- board text removed: "GND_OUT"
- board text removed: "I_1"
- board text removed: "I_2"
- board text removed: "Kelvin"
- board text removed: "PWR_GND"
- board text removed: "Vcc"
